File: Simplified-for-PPT/HF-PA-v10.kicad_sch (KiCad schematic)
At the start: 7 parts, among them Q2 IRF510, T1 Bifilar XFMR, U2 UCC27517DBVR

Commit message: SiC QRO Amplifier
Parts:
- removed R1: 1M / 100K, Resistor_SMD:R_1206_3216Metric_Pad1.30x1.75mm_HandSolder, symbol Device:R
- renumbered C7 to C1, C7 to C2, BNC1 to RF_IN1
Connections:
- net 12V: no longer U2.1 (VDD)
- new net 9v: U2.1 (VDD)
Other:
- note added: "TTL input only!"
- note removed: "8mW to 10mW directly from Si5351"
- moved on the sheet: C1, C2, Q2, RF_IN1, T1, U2
